File: efuse.kicad_sch (KiCad schematic)
At the start: 39 parts, among them IC1 AP7375-50SA-7, IC2 NJM78L12SU3-TE1, IC2 TC74HC08APF, IC3 MLX91220KDC-ABR-050-SP, J21 Conn_01x02_Socket, Q2 TPH4R10ANL, Q3 TPH4R10ANL, Q6 IRFML8244TRPBF, Q7 IRFML8244TRPBF, Q8 IRFML8244TRPBF, U2 TLP785, U3 TLP785

Commit message: コンデンサを追加
Parts:
- added C5: C, Capacitor_SMD:CP_Elec_10x10.5, symbol Device:C
- R11: footprint Resistor_THT:R_Axial_DIN0207_L6.3mm_D2.5mm_P10.16mm_Horizontal -> Resistor_SMD:R_2512_6332Metric
- renumbered IC2 to IC3, Q7 to Q6, Q8 to Q7, Q6 to Q8, R26 to R43, R25 to R44, R24 to R45, R22 to R46, R30 to R47, R23 to R49, R35 to R52, R36 to R53, R12 to R56, R13 to R58, R27 to R59
Connections:
- net GND1: now also C5.2
- net VOUT: now also C5.1

Commit message: 電流センサー変更
Parts:
- removed IC3: MLX91220KDC-ABR-050-SP, Package_SO:SOIC-8_3.9x4.9mm_P1.27mm, symbol SamacSys_Parts:MLX91220KDC-ABR-050-SP
- removed R12, R13, R14, R15, R16, R17: 10kΩ, Resistor_SMD:R_0603_1608Metric, symbol Device:R
- added C11: 0.1μF, Capacitor_SMD:C_0603_1608Metric_Pad1.08x0.95mm_HandSolder, symbol Device:C
- added IC4: ACS711ELCTR-25AB-T, Library:ACS711ELCTR-25AB-T, symbol SamacSys_Parts:ACS711ELCTR-25AB-T
- added R1: 1kΩ, Resistor_SMD:R_0603_1608Metric, symbol Device:R
- added R6: 20kΩ, Resistor_SMD:R_0805_2012Metric, symbol Device:R
- renumbered Q7 to Q10, Q8 to Q11, Q6 to Q9, R43 to R46, R44 to R47, R45 to R48, R46 to R49, R47 to R50, R49 to R52, R52 to R55, R53 to R56, R56 to R59, R58 to R61, R59 to R62
Connections:
- net GND: now also C11.2, IC4.3 (IP-_1), IC4.4 (IP-_2), IC4.5 (GND), R6.2
- net GND1: now also IC4.1 (IP+_1), IC4.2 (IP+_2)
- net Iout: now also IC4.7 (VIOUT), R6.1
- new net +3.3V: C11.1, IC4.8 (VCC), R1.2
- new net FAULT: IC4.6 (~{FAULT}), R1.1
