File: motor.kicad_sch (KiCad schematic)
At the start: 10 parts, among them IC8 DRV8873HPWPRQ1, J2 Conn_01x02_Socket

Commit message: コンデンサを追加
Parts:
- renumbered C26 to C15, C28 to C17, C27 to C18, C25 to C19, C29 to C20, IC8 to IC6, R45 to R5, R43 to R6, R44 to R9

Commit message: 電流センサー変更
Parts:
- renumbered C15 to C16, C17 to C18, C18 to C19, C19 to C20, C20 to C21, R9 to R12, R5 to R8, R6 to R9

Commit message: ESP32バージョン
Parts:
- removed R8: 1.5kΩ, Capacitor_SMD:C_0603_1608Metric_Pad1.08x0.95mm_HandSolder, symbol Device:R
- J2: footprint Connector_AMASS:AMASS_XT30PW-M_1x02_P2.50mm_Horizontal -> Connector_AMASS:AMASS_XT30PW-F_1x02_P2.50mm_Horizontal
Connections:
- net GND1: now also IC6.9 (DISABLE)
- net at IC6.2 (NFAULT), R12.2: now also IC6.11 (NSLEEP)
- net at IC6.10 (IPROPI1), R9.1: now also IC6.12 (IPROPI2)
- net at IC6.14 (OUT2_1), IC6.15 (OUT2_2): now also J2.2 (Pin_2); no longer J2.1 (Pin_1)
- net at IC6.18 (OUT1_1), IC6.19 (OUT1_2): now also J2.1 (Pin_1); no longer J2.2 (Pin_2)
Other:
- moved on the sheet: C19, IC6, R9
